File: CH340T-tryout.kicad_pcb (KiCad board)
At the start: 2 copper layers, 10 parts, among them J1 Conn_01x09, J2 USB_B_Mini, J3 Conn_01x02, U1 CH340T(SSOP20W), Y1 O12M

Commit message: update,
Parts:
- moved J2 13.5 mm to (27.5, 31.5), turned to 180 degrees
- moved Y1 7.99 mm to (35.5, 38.0), turned to 270 degrees
- moved C4 7.40 mm to (32.9, 40.1), turned to 90 degrees
- moved C5 3.60 mm to (32.9, 36.0), turned to 90 degrees
- turned C2 to 90 degrees
Connections:
- net Net-(J1-Pad8) renamed /DTR
- net Net-(J1-Pad9) renamed /RTS
- J1 pad 2: Net-(J1-Pad2) -> /RXD
- J1 pad 3: Net-(J1-Pad3) -> /TXD
- U1 pad 3: Net-(J1-Pad2) -> /TXD
- U1 pad 4: Net-(J1-Pad3) -> /RXD
Routing:
- net GND: track 0.00 -> 54.8 mm
- net +5V: track 0.00 -> 26.6 mm, vias 0 -> 1
- net /DTR: track 0.00 -> 19.0 mm
- net /TXD: track 0.00 -> 14.1 mm
- net /RXD: track 0.00 -> 13.7 mm
- net VCC: track 0.00 -> 12.5 mm
- net Net-(C3-Pad1): track 0.00 -> 10.7 mm, vias 0 -> 1
- net /USB_DP: track 0.00 -> 9.14 mm
- net Net-(C4-Pad2): track 0.00 -> 8.24 mm
- net /USB_DM: track 0.00 -> 8.23 mm
- net Net-(C5-Pad1): track 0.00 -> 7.82 mm
- net /RTS: track 0.00 -> 7.33 mm
- net Net-(J1-Pad7): track 0.00 -> 6.47 mm
- net Net-(J1-Pad6): track 0.00 -> 6.33 mm, vias 0 -> 1
- net Net-(J1-Pad5): track 0.00 -> 5.63 mm
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