File: hardware/CH340T-tryout.kicad_pcb (KiCad board)
At the start: 2 copper layers, 10 parts, among them J1 Conn_01x09, J2 USB_B_Mini, J3 Conn_01x02, U1 CH340T(SSOP20W), Y1 O12M

Commit message: update,
Parts:
- removed J2: USB_B_Mini, Connector_USB:USB_Micro-B_Molex_47346-0001
- removed J3: Conn_01x02, Connector_PinHeader_1.27mm:PinHeader_1x02_P1.27mm_Vertical
- added C6: C22pf,0603, Capacitor_SMD:C_0603_1608Metric_Pad1.05x0.95mm_HandSolder, F.Cu at (26.5, 31.5)
- added U2: USB_Micro, footprint-lib:USB_Micro-B_Molex-105017-0001, F.Cu at (36.2, 23.2)
- C1: value C226,6.3v,0603 -> C475,0603
- C2: value C104,0603 -> C225,0603
- C3: value C102,0603 -> C104,0603
- C4: value C22pf,0603 -> C103,0603
- C5: moved to F.Cu
- J1: value Conn_01x09 -> Conn_01x04_Female; footprint Connector_PinHeader_1.27mm:PinHeader_1x09_P1.27mm_Vertical -> Connector_PinHeader_1.27mm:PinHeader_1x10_P1.27mm_Vertical; moved to F.Cu
- U1: value CH340T(SSOP20W) -> CH340T; footprint Package_SO:SSOP-20_5.3x7.2mm_P0.65mm -> footprint-lib:CH340T_SSOP-20
- Y1: value O12M -> O_12M,3225; footprint w_crystal:crystal_hc-49s -> footprint-lib:OSC_3225
- moved J1 27.3 mm to (46.2, 27.5), turned to 0 degrees
- moved C1 15.3 mm to (36.0, 30.0)
- moved U1 11.3 mm to (36.4, 32.5), turned to 0 degrees
- moved C3 10.1 mm to (36.0, 31.8), turned to 0 degrees
- moved C2 9.66 mm to (36.0, 35.5), turned to 0 degrees
- moved Y1 9.46 mm to (26.5, 35.0), turned to 90 degrees
- moved C4 7.29 mm to (36.0, 33.5), turned to 0 degrees
- moved C5 6.88 mm to (26.5, 38.5), turned to 180 degrees
Connections:
- C1 pad 2: VCC -> +5V
- C2 pad 1: VCC -> +5V
- C3 pad 1: Net-(C3-Pad1) -> +5V
- C4 pad 1: GND -> Net-(C4-Pad1)
- C4 pad 2: Net-(C4-Pad2) -> GND
- J1 pad 2: /RXD -> +5V
- J1 pad 3: /TXD -> Net-(J1-Pad3)
- J1 pad 8: /DTR -> Net-(J1-Pad8)
- J1 pad 9: /RTS -> Net-(J1-Pad9)
- U1 pad 1: Net-(U1-Pad1) -> (no net)
- U1 pad 10: Net-(C5-Pad1) -> Net-(C6-Pad1)
- U1 pad 11: Net-(J1-Pad4) -> Net-(J1-Pad8)
- U1 pad 12: Net-(J1-Pad5) -> Net-(J1-Pad7)
- U1 pad 14: Net-(J1-Pad7) -> Net-(J1-Pad5)
- U1 pad 15: /DTR -> Net-(J1-Pad4)
- U1 pad 16: /RTS -> Net-(J1-Pad3)
- U1 pad 17: Net-(U1-Pad17) -> (no net)
- U1 pad 18: Net-(U1-Pad18) -> (no net)
- U1 pad 19: VCC -> +5V
- U1 pad 2: Net-(U1-Pad2) -> (no net)
- U1 pad 20: Net-(U1-Pad20) -> (no net)
- U1 pad 3: /TXD -> Net-(J1-Pad10)
- U1 pad 4: /RXD -> Net-(J1-Pad9)
- U1 pad 5: Net-(C3-Pad1) -> Net-(C4-Pad1)
- U1 pad 6: /USB_DP -> Net-(U1-Pad6)
- U1 pad 7: /USB_DM -> Net-(U1-Pad7)
- U1 pad 9: Net-(C4-Pad2) -> Net-(C5-Pad1)
- Y1 pad 2: Net-(C4-Pad2) -> GND
Routing:
- net Net-(J1-Pad10): track 0.00 -> 41.5 mm
- net Net-(J1-Pad9): track 0.00 -> 40.4 mm
- net /DTR: track 19.0 -> 0.00 mm
- net Net-(C6-Pad1): track 0.00 -> 18.8 mm
- net +5V: track 26.6 -> 41.4 mm, vias 1 -> 0
- net /TXD: track 14.1 -> 0.00 mm
- net /RXD: track 13.7 -> 0.00 mm
- net VCC: track 12.5 -> 0.00 mm
- net Net-(U1-Pad7): track 0.00 -> 11.2 mm
- net Net-(C3-Pad1): track 10.7 -> 0.00 mm, vias 1 -> 0
- net Net-(U1-Pad6): track 0.00 -> 10.3 mm
- net /USB_DP: track 9.14 -> 0.00 mm
- net Net-(C4-Pad2): track 8.24 -> 0.00 mm
- net /USB_DM: track 8.23 -> 0.00 mm
- net GND: track 54.8 -> 46.9 mm
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
Commit message: update,
Parts:
- J1: value Conn_01x04_Female -> SERIAL_HEADER
Connections:
- net Net-(J1-Pad10) renamed /TXD
- net Net-(J1-Pad3) renamed /RTS
- net Net-(J1-Pad4) renamed /DTR
- net Net-(J1-Pad5) renamed /DCD
- net Net-(J1-Pad6) renamed /RI
- net Net-(J1-Pad7) renamed /DSR
- net Net-(J1-Pad8) renamed /CTS
- net Net-(J1-Pad9) renamed /RXD
- net Net-(U1-Pad6) renamed /USB_P
- net Net-(U1-Pad7) renamed /USB_N
- U2 pad 5: (no net) -> GND
- U2 pad 6: Net-(U2-Pad6) -> GND
- U2 pad 7: Net-(U2-Pad7) -> GND
- U2 pad 8: (no net) -> GND
- U2 pad 9: (no net) -> GND
Routing:
- net GND: track 46.9 -> 68.8 mm, vias 0 -> 1
- net /RXD: track 40.4 -> 23.9 mm, vias 0 -> 1
- net /TXD: track 41.5 -> 27.7 mm, vias 0 -> 1
- net +5V: track 41.4 -> 29.9 mm, vias 0 -> 2
- net Net-(U2-Pad7): track 5.05 -> 0.00 mm
- net Net-(U2-Pad6): track 5.05 -> 0.00 mm
