File: hardware/CH340T-tryout.sch (KiCad schematic (older format))
At the start: 10 parts

Commit message: update,
Parts:
- J1: renamed from J?; footprint (none) -> Connector_PinHeader_1.27mm:PinHeader_1x10_P1.27mm_Vertical
- gave numbers to parts that had none: 9
Changed lines of the file:
@@
 $EndDescr
 $Comp
-L taobao-components:USB_Micro U?
+L taobao-components:USB_Micro U2
 U 1 1 5D058DA8
 P 2100 2300
-F 0 "U?" H 2100 2765 50  0000 C CNN
+F 0 "U2" H 2100 2765 50  0000 C CNN
 F 1 "USB_Micro" H 2100 2674 50  0000 C CNN
 F 2 "footprint-lib:USB_Micro-B_Molex-105017-0001" H 2100 1800 50  0001 C CNN
@@
 $EndComp
 $Comp
-L taobao-components:CH340T U?
+L taobao-components:CH340T U1
 U 1 1 5D05D663
 P 4900 2150
-F 0 "U?" H 4875 3093 60  0000 C CNN
+F 0 "U1" H 4875 3093 60  0000 C CNN
 F 1 "CH340T" H 4875 2987 60  0000 C CNN
 F 2 "footprint-lib:CH340T_SSOP-20" H 4875 2881 60  0000 C CNN
@@
 $EndComp
 $Comp
-L taobao-osc:O_12M,3225 Y?
+L taobao-osc:O_12M,3225 Y1
 U 1 1 5D05E9C1
 P 3600 2700
-F 0 "Y?" H 3600 2925 50  0000 C CNN
+F 0 "Y1" H 3600 2925 50  0000 C CNN
 F 1 "O_12M,3225" H 3600 2834 50  0000 C CNN
 F 2 "footprint-lib:OSC_3225" H 3600 2700 50  0001 C CNN
@@
 	3400 2700 3500 2700
 $Comp
-L taobao-c:C22pf,0603 C?
+L taobao-c:C22pf,0603 C5
 U 1 1 5D061A62
 P 3400 2900
-F 0 "C?" H 3492 2946 50  0000 L CNN
+F 0 "C5" H 3492 2946 50  0000 L CNN
 F 1 "C22pf,0603" H 3492 2855 50  0000 L CNN
 F 2 "Capacitor_SMD:C_0603_1608Metric_Pad1.05x0.95mm_HandSolder" H 3400 2900 50  0001 C CNN
@@
 $EndComp
 $Comp
-L taobao-c:C22pf,0603 C?
+L taobao-c:C22pf,0603 C6
 U 1 1 5D06326C
 P 3850 2900
-F 0 "C?" H 3942 2946 50  0000 L CNN
+F 0 "C6" H 3942 2946 50  0000 L CNN
 F 1 "C22pf,0603" H 3942 2855 50  0000 L CNN
 F 2 "Capacitor_SMD:C_0603_1608Metric_Pad1.05x0.95mm_HandSolder" H 3850 2900 50  0001 C CNN
@@
 Connection ~ 3400 2700
 $Comp
-L power:GND #PWR?
+L power:GND #PWR0101
 U 1 1 5D0658C0
 P 3650 3200
-F 0 "#PWR?" H 3650 2950 50  0001 C CNN
+F 0 "#PWR0101" H 3650 2950 50  0001 C CNN
 F 1 "GND" H 3655 3027 50  0000 C CNN
 F 2 "" H 3650 3200 50  0001 C CNN
@@
 	3550 3100 3650 3100
 $Comp
-L taobao-c:C103,0603 C?
+L taobao-c:C103,0603 C4
 U 1 1 5D06DB24
 P 3950 1850
-F 0 "C?" H 4042 1896 50  0000 L CNN
+F 0 "C4" H 4042 1896 50  0000 L CNN
 F 1 "C103,0603" H 4042 1805 50  0000 L CNN
 F 2 "Capacitor_SMD:C_0603_1608Metric_Pad1.05x0.95mm_HandSolder" H 3950 1850 50  0001 C CNN
@@
 $EndComp
 $Comp
-L taobao-c:C104,0603 C?
+L taobao-c:C104,0603 C3
 U 1 1 5D06F240
 P 3450 1850
-F 0 "C?" H 3542 1896 50  0000 L CNN
+F 0 "C3" H 3542 1896 50  0000 L CNN
 F 1 "C104,0603" H 3542 1805 50  0000 L CNN
 F 2 "Capacitor_SMD:C_0603_1608Metric_Pad1.05x0.95mm_HandSolder" H 3450 1850 50  0001 C CNN
@@
 $EndComp
 $Comp
-L taobao-c:C225,0603 C?
+L taobao-c:C225,0603 C2
 U 1 1 5D06FAA1
 P 3200 1850
-F 0 "C?" H 3292 1896 50  0000 L CNN
+F 0 "C2" H 3292 1896 50  0000 L CNN
 F 1 "C225,0603" H 3292 1805 50  0000 L CNN
 F 2 "Capacitor_SMD:C_0603_1608Metric_Pad1.05x0.95mm_HandSolder" H 3200 1850 50  0001 C CNN
@@
 Connection ~ 3450 2000
 $Comp
-L power:GND #PWR?
+L power:GND #PWR0102
 U 1 1 5D0758C8
 P 3650 2050
-F 0 "#PWR?" H 3650 1800 50  0001 C CNN
+F 0 "#PWR0102" H 3650 1800 50  0001 C CNN
 F 1 "GND" H 3655 1877 50  0000 C CNN
 F 2 "" H 3650 2050 50  0001 C CNN
@@
 	3950 1700 3950 1750
 $Comp
-L Connector:Conn_01x10_Female J?
+L Connector:Conn_01x10_Female J1
 U 1 1 5D097AD0
 P 6500 2100
-F 0 "J?" H 6392 1375 50  0000 C CNN
+F 0 "J1" H 6392 1375 50  0000 C CNN
 F 1 "Conn_01x04_Female" H 6392 1466 50  0000 C CNN
-F 2 "" H 6500 2100 50  0001 C CNN
+F 2 "Connector_PinHeader_1.27mm:PinHeader_1x10_P1.27mm_Vertical" H 6500 2100 50  0001 C CNN
 F 3 "~" H 6500 2100 50  0001 C CNN
 	1    6500 2100
@@
 	5500 1700 6300 1700
 $Comp
-L power:+5V #PWR?
+L power:+5V #PWR0103
 U 1 1 5D0A14B8
 P 2850 1450
-F 0 "#PWR?" H 2850 1300 50  0001 C CNN
+F 0 "#PWR0103" H 2850 1300 50  0001 C CNN
 F 1 "+5V" H 2865 1623 50  0000 C CNN
 F 2 "" H 2850 1450 50  0001 C CNN
@@
 Connection ~ 2850 1600
 $Comp
-L power:+5V #PWR?
+L power:+5V #PWR0104
 U 1 1 5D0A9573
 P 4550 1050
-F 0 "#PWR?" H 4550 900 50  0001 C CNN
+F 0 "#PWR0104" H 4550 900 50  0001 C CNN
 F 1 "+5V" V 4565 1178 50  0000 L CNN
 F 2 "" H 4550 1050 50  0001 C CNN
@@
 $EndComp
 $Comp
-L power:GND #PWR?
+L power:GND #PWR0105
 U 1 1 5D0A9D8F
 P 5150 1050
-F 0 "#PWR?" H 5150 800 50  0001 C CNN
+F 0 "#PWR0105" H 5150 800 50  0001 C CNN
 F 1 "GND" V 5155 922 50  0000 R CNN
 F 2 "" H 5150 1050 50  0001 C CNN
@@
 $EndComp
 $Comp
-L taobao-c:C475,0603 C?
+L taobao-c:C475,0603 C1
 U 1 1 5D0AA385
 P 4850 1050
-F 0 "C?" V 4621 1050 50  0000 C CNN
+F 0 "C1" V 4621 1050 50  0000 C CNN
 F 1 "C475,0603" V 4712 1050 50  0000 C CNN
 F 2 "Capacitor_SMD:C_0603_1608Metric_Pad1.05x0.95mm_HandSolder" H 4850 1050 50  0001 C CNN
@@
 	6300 2400 6050 2400
 $Comp
-L power:+5V #PWR?
+L power:+5V #PWR0106
 U 1 1 5D0A562E
 P 6050 2750
-F 0 "#PWR?" H 6050 2600 50  0001 C CNN
+F 0 "#PWR0106" H 6050 2600 50  0001 C CNN
 F 1 "+5V" H 6065 2923 50  0000 C CNN
 F 2 "" H 6050 2750 50  0001 C CNN
@@
 	6200 2700 6200 2500
 $Comp
-L power:GND #PWR?
+L power:GND #PWR0107
 U 1 1 5D09B4B9
 P 6200 2700
-F 0 "#PWR?" H 6200 2450 50  0001 C CNN
+F 0 "#PWR0107" H 6200 2450 50  0001 C CNN
 F 1 "GND" H 6205 2527 50  0000 C CNN
 F 2 "" H 6200 2700 50  0001 C CNN

Commit message: update,
Connections:
- net GND: now also U2.5 (GND), U2.6 (MH1), U2.7 (MH2), U2.8 (MH3), U2.9 (MH4)
- no-connect marks 0 -> 3
Changed lines of the file:
@@
 EndData
 $EndBitmap
+$Comp
+L power:GND #PWR0108
+U 1 1 5D0516E0
+P 1550 2750
+F 0 "#PWR0108" H 1550 2500 50  0001 C CNN
+F 1 "GND" H 1555 2577 50  0000 C CNN
+F 2 "" H 1550 2750 50  0001 C CNN
+F 3 "" H 1550 2750 50  0001 C CNN
+	1    1550 2750
+	1    0    0    -1
+$EndComp
+Wire Wire Line
+	1700 2100 1550 2100
+Wire Wire Line
+	1550 2100 1550 2200
+Wire Wire Line
+	1700 2200 1550 2200
+Connection ~ 1550 2200
+Wire Wire Line
+	1550 2200 1550 2400
+Wire Wire Line
+	1700 2400 1550 2400
+Connection ~ 1550 2400
+Wire Wire Line
+	1550 2400 1550 2500
+Wire Wire Line
+	1700 2500 1550 2500
+Connection ~ 1550 2500
+Wire Wire Line
+	1550 2500 1550 2750
+$Comp
+L power:GND #PWR0109
+U 1 1 5D057019
+P 2650 2750
+F 0 "#PWR0109" H 2650 2500 50  0001 C CNN
+F 1 "GND" H 2655 2577 50  0000 C CNN
+F 2 "" H 2650 2750 50  0001 C CNN
+F 3 "" H 2650 2750 50  0001 C CNN
+	1    2650 2750
+	1    0    0    -1
+$EndComp
+Wire Wire Line
+	2500 2500 2650 2500
+Wire Wire Line
+	2650 2500 2650 2750
+NoConn ~ 2500 2400
+NoConn ~ 5500 2600
+NoConn ~ 5500 2700
 $EndSCHEMATC

Commit message: update,
Parts:
- J1: value Conn_01x04_Female -> SERIAL_HEADER
Connections:
- net USB_N: now reaches U1.7 (UD-), U2.2 (D-)
- net USB_P: now reaches U1.6 (UD+), U2.3 (D+)
- net CTS: now reaches J1.8 (Pin_8), U1.11 (CTS#)
- net DSR: now reaches J1.7 (Pin_7), U1.12 (DSR#)
- net RI: now reaches J1.6 (Pin_6), U1.13 (RI#)
- net DCD: now reaches J1.5 (Pin_5), U1.14 (DCD#)
- net DTR: now reaches J1.4 (Pin_4), U1.15 (DTR#)
- net RTS: now reaches J1.3 (Pin_3), U1.16 (RTS#)
- net TXD: now reaches J1.10 (Pin_10), U1.3 (TXD)
- net RXD: now reaches J1.9 (Pin_9), U1.4 (RXD)
Changed lines of the file:
@@
 F 0 "U1" H 4875 3093 60  0000 C CNN
 F 1 "CH340T" H 4875 2987 60  0000 C CNN
-F 2 "footprint-lib:CH340T_SSOP-20" H 4875 2881 60  0000 C CNN
+F 2 "footprint-lib:CH340T_SSOP-20" H 4875 2881 60  0001 C CNN
 F 3 "" H 4900 2150 60  0000 C CNN
 	1    4900 2150
@@
 P 6500 2100
 F 0 "J1" H 6392 1375 50  0000 C CNN
-F 1 "Conn_01x04_Female" H 6392 1466 50  0000 C CNN
+F 1 "SERIAL_HEADER" H 6392 1466 50  0000 C CNN
 F 2 "Connector_PinHeader_1.27mm:PinHeader_1x10_P1.27mm_Vertical" H 6500 2100 50  0001 C CNN
 F 3 "~" H 6500 2100 50  0001 C CNN
@@
 NoConn ~ 5500 2600
 NoConn ~ 5500 2700
+Text Label 3100 2200 2    50   ~ 0
+USB_N
+Text Label 3100 2300 2    50   ~ 0
+USB_P
+Text Label 6200 1600 2    50   ~ 0
+TXD
+Text Label 6200 1700 2    50   ~ 0
+RXD
+Text Label 6200 1800 2    50   ~ 0
+CTS
+Text Label 6200 1900 2    50   ~ 0
+DSR
+Text Label 6200 2000 2    50   ~ 0
+RI
+Text Label 6200 2100 2    50   ~ 0
+DCD
+Text Label 6200 2200 2    50   ~ 0
+DTR
+Text Label 6200 2300 2    50   ~ 0
+RTS
 $EndSCHEMATC

Commit message: update,
Parts:
- added JP1: SLEEP_EN, Jumper:SolderJumper-2_P1.3mm_Open_RoundedPad1.0x1.5mm, symbol my_solder_jumper:SolderJumper_2_Open_round
Connections:
- net GND: now also JP1.2 (B)
- net at U1.20 (NOS#): now also JP1.1 (A)
- no-connect marks 3 -> 2
